Commit message: Add mapping and localization simulation flow

File: urdf/mobile_manipulator.urdf (robot description, URDF)
Before this commit: robot mobile_manipulator, 14 links, 13 joints
Links:
- added link lidar_link, mass 0.25; collision cylinder length=0.08 radius=0.07; visual cylinder length=0.08 radius=0.07
- added link sensor_mount_link, mass 0.35; collision box size=0.16 0.12 0.08; visual box size=0.16 0.12 0.08
- link left_forearm_link: geometry collision cylinder length=0.30 radius=0.04; visual cylinder length=0.30 radius=0.04
- link left_upper_arm_link: geometry collision cylinder length=0.34 radius=0.045; visual cylinder length=0.34 radius=0.045
- link right_forearm_link: geometry collision cylinder length=0.30 radius=0.04; visual cylinder length=0.30 radius=0.04
- link right_upper_arm_link: geometry collision cylinder length=0.34 radius=0.045; visual cylinder length=0.34 radius=0.045
Joints:
- added joint lidar_fixed_joint: type fixed, parent sensor_mount_link, child lidar_link, origin xyz=0.02 0 0.08
- added joint sensor_mount_fixed_joint: type fixed, parent head_sensor_link, child sensor_mount_link, origin xyz=0.16 0 0.10
- joint left_elbow_joint: origin xyz=0 0.42 0 -> xyz=0 0 -0.34
- joint left_hand_fixed_joint: origin xyz=0 0.39 0 -> xyz=0 0 -0.32
- joint right_elbow_joint: origin xyz=0 -0.42 0 -> xyz=0 0 -0.34
- joint right_hand_fixed_joint: origin xyz=0 -0.39 0 -> xyz=0 0 -0.32

Commit message: Add Nav2 navigation and safety shell visualization updates

File: urdf/mobile_manipulator.urdf (robot description, URDF)
Before this commit: robot mobile_manipulator, 16 links, 15 joints
Joints:
- joint left_shoulder_yaw_joint: origin xyz=0 0.22 0.25 -> xyz=0 0.22 0.25 rpy=1.57079632679 0 0
- joint right_shoulder_yaw_joint: origin xyz=0 -0.22 0.25 -> xyz=0 -0.22 0.25 rpy=-1.57079632679 0 0
